File: WizzardCartRPack.kicad_pcb (KiCad board)
At the start: 2 copper layers, 72.7 x 54.5 mm, 7 parts, among them SW1 SW_DIP_x05, U1 27C801

Commit message: Add files via upload
Added THIS SIDE UP and mounting holes.
Parts:
- added REF**: MountingHole_3.2mm_M3, MountingHole:MountingHole_3.2mm_M3, F.Cu at (143.2, 120.6)
- added REF**: MountingHole_3.2mm_M3, MountingHole:MountingHole_3.2mm_M3, F.Cu at (103.8, 78.8)
Other:
- board text added: "THIS SIDE UP"

Commit message: Add files via upload
Updated to KiCAD 6.
Parts:
- removed REF** (x2): MountingHole_3.2mm_M3, MountingHole:MountingHole_3.2mm_M3
- removed RN1: 4.7k, Resistor_THT:R_Array_SIP7
- added R1: 4.7k, Resistor_THT:R_Axial_DIN0204_L3.6mm_D1.6mm_P7.62mm_Horizontal, F.Cu at (136.7, 122.4)
- added R2: 4.7k, Resistor_THT:R_Axial_DIN0204_L3.6mm_D1.6mm_P7.62mm_Horizontal, F.Cu at (132.9, 122.4)
- added R3: 4.7k, Resistor_THT:R_Axial_DIN0204_L3.6mm_D1.6mm_P7.62mm_Horizontal, F.Cu at (129.1, 122.4)
- added R4: 4.7k, Resistor_THT:R_Axial_DIN0204_L3.6mm_D1.6mm_P7.62mm_Horizontal, F.Cu at (125.2, 122.4)
- added R5: 4.7k, Resistor_THT:R_Axial_DIN0204_L3.6mm_D1.6mm_P7.62mm_Horizontal, F.Cu at (121.5, 122.4)
- added R6: 4.7k, Resistor_THT:R_Axial_DIN0204_L3.6mm_D1.6mm_P7.62mm_Horizontal, F.Cu at (104.2, 80.5)
- E1: footprint CheshBits:36Edge -> WizzardCart:36Edge
Routing:
- net Net-(D1-Pad2): track 72.0 -> 25.3 mm
- net Net-(R5-Pad2): track 43.0 -> 25.7 mm
- net Net-(R4-Pad2): track 60.6 -> 49.6 mm
- net Net-(R1-Pad2): track 40.9 -> 51.4 mm
- net Net-(R3-Pad2): track 56.4 -> 51.4 mm
- net Net-(R2-Pad2): track 81.6 -> 83.7 mm
- net +5V: track 115.0 -> 116.5 mm
Other:
- net class Default removed
- net class Power removed
- board text removed: "THIS SIDE UP"
