File: WizzardCartRPack.sch (KiCad schematic (older format))
At the start: 7 parts, among them SW1 SW_DIP_x05, U1 27C801

Commit message: Add files via upload
Updated to KiCAD 6.
Parts:
- removed E1: 36Edge, CheshBits:36Edge, symbol EdgeConnector:36Edge
- added E1: 36Edge, WizzardCart:36Edge, symbol WizzardCart-rescue:36Edge-EdgeConnector
Connections:
- net +5V: now also E1.1 (+5v)
- net GND: now also E1.35 (GND)
- net at U1.10 (A2): now also E1.9 (A2)
- net at U1.11 (A1): now also E1.12 (A1)
- net at U1.12 (A0): now also E1.11 (A0)
- net at U1.13 (D0): now also E1.22 (D0)
- net at U1.14 (D1): now also E1.21 (D1)
- net at U1.15 (D2): now also E1.20 (D2)
- net at U1.17 (D3): now also E1.19 (D3)
- net at U1.18 (D4): now also E1.23 (D4)
- net at U1.19 (D5): now also E1.24 (D5)
- net at U1.20 (D6): now also E1.25 (D6)
- net at U1.21 (D7): now also E1.28 (D7)
- net at U1.23 (A10): now also E1.14 (A10)
- net at U1.25 (A11): now also E1.13 (A11)
- net at U1.26 (A9): now also E1.4 (A9)
- net at U1.27 (A8): now also E1.3 (A8)
- net at U1.28 (A13): now also E1.15 (A13)
- net at U1.29 (A14): now also E1.18 (A14)
- net at U1.4 (A12): now also E1.16 (A12)
- net at U1.5 (A7): now also E1.6 (A7)
- net at U1.6 (A6): now also E1.5 (A6)
- net at U1.7 (A5): now also E1.8 (A5)
- net at U1.8 (A4): now also E1.7 (A4)
- net at U1.9 (A3): now also E1.10 (A3)
- net at D1.1 (K): now also E1.29 (_ROM1)
- net at D2.1 (K): now also E1.32 (_ROM2)
- new net: E1.33 (_ROM0), E1.34 (_ROMR)
Changed lines of the file:
@@
 	1    0    0    -1
 $EndComp
+$Comp
+L WizzardCart-rescue:36Edge-EdgeConnector E1
+U 1 1 5F317394
+P 4400 6450
+F 0 "E1" H 4335 6647 50  0000 C CNN
+F 1 "36Edge" H 4335 6556 50  0000 C CNN
+F 2 "WizzardCart:36Edge" H 4335 6465 50  0000 C CNN
+F 3 "" H 4400 6450 50  0001 C CNN
+	1    4400 6450
+	1    0    0    1
+$EndComp
+Wire Wire Line
+	2600 6000 2600 5150
 Wire Wire Line
 	2600 1050 5800 1050
@@
 	3500 2200 5400 2200
 Wire Wire Line
+	3200 6000 3200 2300
+Wire Wire Line
 	3200 2300 5400 2300
 Wire Wire Line
+	3300 6000 3300 2400
+Wire Wire Line
 	3300 2400 5400 2400
 Wire Wire Line
+	3000 6000 3000 2500
+Wire Wire Line
 	3000 2500 5400 2500
 Wire Wire Line
+	3100 6000 3100 2600
+Wire Wire Line
 	3100 2600 5400 2600
 Wire Wire Line
+	2800 6000 2800 2700
+Wire Wire Line
 	2800 2700 5400 2700
+Wire Wire Line
+	2900 6000 2900 2800
 Wire Wire Line
 	2900 2800 5400 2800
@@
 Wire Wire Line
 	2300 4500 4700 4500
-$Comp
-L EdgeConnector:36Edge E1
-U 1 1 5F5C15F3
-P 4400 5550
-F 0 "E1" H 4335 5747 50  0000 C CNN
-F 1 "36Edge" H 4335 5656 50  0000 C CNN
-F 2 "CheshBits:36Edge" H 4335 5565 50  0000 C CNN
-F 3 "" H 4400 5550 50  0001 C CNN
-	1    4400 5550
-	1    0    0    -1
-$EndComp
-Wire Wire Line
-	3300 6000 3300 2400
-Wire Wire Line
-	3200 6000 3200 2300
-Wire Wire Line
-	3100 6000 3100 2600
-Wire Wire Line
-	3000 6000 3000 2500
-Wire Wire Line
-	2900 6000 2900 2800
-Wire Wire Line
-	2800 6000 2800 2700
-Wire Wire Line
-	2600 6000 2600 5150
 $EndSCHEMATC
